File: Ver-01.xx/KiCad/Controller_Bluetooth.kicad_sch (KiCad schematic)
At the start: 21 parts, among them J1 LOETJUMPER, K15 Stiftleiste_1x06, U1 RN4678, X1 STM32F405VGT, Y1 Crystal

Commit message: After production test
Footprint D1 and Y1 changed.
LED shunt R=330
Parts:
- Y1: footprint Crystal:Crystal_SMD_5032-2Pin_5.0x3.2mm -> Crystal:Crystal_SMD_Abracon_ABM3-2Pin_5.0x3.2mm
Changed lines of the file:
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@@
       (effects (font (size 1.27 1.27)) (justify right))
     )
-    (property "Footprint" "Crystal:Crystal_SMD_5032-2Pin_5.0x3.2mm" (at 33.02 24.13 0)
+    (property "Footprint" "Crystal:Crystal_SMD_Abracon_ABM3-2Pin_5.0x3.2mm" (at 33.02 24.13 0)
       (effects (font (size 1.27 1.27)) hide)
     )
